File: electronics/radiohead-sys/audio.kicad_sch (KiCad schematic)
At the start: 0 parts

Commit message: completing all major schematics, just need to add usb devices
Parts:
- added LS1, LS2: 8ohm, symbol Device:Speaker
- added U1, U2: MAX98357A, Package_DFN_QFN:TQFN-16-1EP_3x3mm_P0.5mm_EP1.23x1.23mm, symbol Audio:MAX98357A
Connections:
- new net: LS1.2, U1.10 (OUTN)
- new net: LS1.1, U1.9 (OUTP)
- new net: LS2.2, U2.10 (OUTN)
- new net: LS2.1, U2.9 (OUTP)
- new net GND: U1.11 (GND), U1.15 (GND), U1.2 (GAIN_SLOT), U1.3 (GND), U2.11 (GND), U2.15 (GND), U2.2 (GAIN_SLOT), U2.3 (GND)
- new net SPEAKER.J41.I2S4.LRCK: U1.14 (LRCLK), U2.14 (LRCLK)
- new net SPEAKER.J41.I2S4.SCLK: U1.16 (BCLK), U2.16 (BCLK)
- new net SPEAKER.J41.I2S4.SDIN: U1.1 (DIN), U2.1 (DIN)
- new net SPEAKER.J41.I2S4.SDOUT: U1.4 (~{SD_MODE}), U2.4 (~{SD_MODE})
- new net VDD: U1.7 (VDD), U1.8 (VDD), U2.7 (VDD), U2.8 (VDD)
- no-connect marks 0 -> 2
Other:
- note added: "+12dB"
- note added: "Resources - https://learn.sparkfun.com/tutorials/i2s-audio-breakout-hookup-guide - https://www.sparkfun.com/wide-frequency-range-speaker-3in-polypropylene-cone.html"
- note added: "SPARK.COM-18379 Note: - 8 ohm Imp., 10W Cont. - This will likely need amplification/power increase from I2S chip - I don't know if we can drive two MAX98357A from the same I2S source"
- note added: "VDD = 2v5-5v5 Note: - I2S amplifier delivers up to 3.2W power into a 4ohm load - Pretend this is Sparkfun breakout for same chip"
- company: (none) -> Alexander Adranly
- title: (none) -> Speaker System
